Commit message: added new test urdf, updated diffbot_controllers to match new urdf

File: description/ros2_control/diffbot.ros2_control.xacro (robot description, xacro)
@@ -1,5 +1,5 @@
 <?xml version="1.0"?>
 <robot xmlns:xacro="http://www.ros.org/wiki/xacro">
-  <xacro:macro name="diffbot_ros2_control" params="name prefix use_mock_hardware">
+  <xacro:macro name="diffbot_ros2_control" params="name use_mock_hardware">
     <ros2_control name="${name}" type="system">
       <xacro:unless value="${use_mock_hardware}">
@@ -20,20 +20,20 @@
         </hardware>
       </xacro:if>
-      <joint name="${prefix}front_left_wheel_joint">
+      <joint name="front_left_wheel_joint">
         <command_interface name="velocity"/>
         <state_interface name="position"/>
         <state_interface name="velocity"/>
       </joint>
-      <joint name="${prefix}front_right_wheel_joint">
+      <joint name="front_right_wheel_joint">
         <command_interface name="velocity"/>
         <state_interface name="position"/>
         <state_interface name="velocity"/>
       </joint>
-      <joint name="${prefix}back_left_wheel_joint">
+      <joint name="back_left_wheel_joint">
         <command_interface name="velocity"/>
         <state_interface name="position"/>
         <state_interface name="velocity"/>
       </joint>
-      <joint name="${prefix}back_right_wheel_joint">
+      <joint name="back_right_wheel_joint">
         <command_interface name="velocity"/>
         <state_interface name="position"/>

File: description/urdf/diffbot.urdf.xacro (robot description, xacro)
@@ -11,4 +11,4 @@
   <xacro:diffbot prefix="$(arg prefix)" />
   <xacro:diffbot_ros2_control
-    name="DiffBot" prefix="$(arg prefix)" use_mock_hardware="$(arg use_mock_hardware)"/>
+    name="DiffBot" use_mock_hardware="$(arg use_mock_hardware)"/>
 </robot>
